File: MRCS-Optical-Detector.brd (EAGLE design)
At the start: 45.6 x 30.3 mm, 17 parts, among them IC1 LM2903N, T1 PT19, T2 2N4401

Commit message: fixed invalid XML names (cap with ',' in name)
Parts:
- C1: device rcl:E2,5-5 -> rcl:E2.5-5
Changed lines of the file:
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@@
 <attribute name="VALUE" x="37.338" y="15.621" size="0.8128" layer="21" font="vector" ratio="15" rot="R180"/>
 </element>
-<element name="C1" library="rcl" package="E2,5-5" value="1 uF Tant" x="22.86" y="10.414" smashed="yes" rot="MR0">
+<element name="C1" library="rcl" package="E2.5-5" value="1 uF Tant" x="22.86" y="10.414" smashed="yes" rot="MR0">
 <attribute name="NAME" x="22.225" y="11.811" size="1.27" layer="21" ratio="10"/>
 <attribute name="VALUE" x="20.447" y="8.001" size="1.27" layer="27" ratio="10"/>
